Commit message: FIX ABB 6700 + tracks,  robot orientation

File: robot_files/abb_irb_6700_track_irtb_6004/4_urdfs/abb_irbt6004_670_support/urdf/abb_irb6700_175_305_ibois_tworobots.xacro (robot description, xacro)
@@ -12,5 +12,5 @@
       <parent link="world" />
       <child link = "rob2_axis" />
-      <origin xyz="0.0 3.0 0.0" rpy="0.0 0.0 0.0" />
+      <origin xyz="0.0 3.0 0.0" rpy="0.0 0.0 	3.14159265358979323846" />
   </joint>
   <xacro:abb_irb6700_175_305_ibois prefix="rob2_" />

File: robot_files/abb_irb_6700_track_irtb_6004_2x/4_urdfs/abb_irbt6004_670_support/urdf/abb_irb6700_175_305_ibois_tworobots.xacro (robot description, xacro)
@@ -1,17 +1,19 @@
 <?xml version="1.0"?>
 <robot name="abb_irb6700_175_305_ibois" xmlns:xacro="http://ros.org/wiki/xacro">
+  <!--linking another xacro file of the robot without rail-->
   <xacro:include filename="$(find abb_irbt6004_670_support)/urdf/abb_irb6700_175_305_ibois_macro.xacro"/>
+  <xacro:include filename="$(find abb_irbt6004_670_support)/urdf/abb_irb6700_175_305_crcl_macro.xacro"/>
   <link name="world" />
   <joint name="world_joint1" type="fixed">
       <parent link="world" />
       <child link = "rob1_axis" />
-      <origin xyz="0.0 0.0 0.0" rpy="0.0 0.0 0.0" />
+      <origin xyz="0 -1.5 0.0" rpy="0.0 0.0 0.0" /> <!--translation of the track-->
   </joint>
-  <xacro:abb_irb6700_175_305_ibois prefix="rob1_" />
+  <xacro:abb_irb6700_175_305_ibois prefix="rob1_" /> <!--robot with different base rotation-->
   <joint name="world_joint2" type="fixed">
       <parent link="world" />
       <child link = "rob2_axis" />
-      <origin xyz="0.0 3.0 0.0" rpy="0.0 0.0 0.0" />
+      <origin xyz="0 1.5 0.0" rpy="0.0 0.0 0" /> <!--translation of the track-->
   </joint>
-  <xacro:abb_irb6700_175_305_ibois prefix="rob2_" />
+  <xacro:abb_irb6700_175_305_crcl prefix="rob2_" /> <!--robot with different base rotation-->
 </robot>

File: robot_files/abb_irb_6700_track_irtb_6004_2x/4_urdfs/abb_irbt6004_670_support/urdf/abb_irbt6004_670.xacro (robot description, xacro)
@@ -8,5 +8,5 @@
       </inertial>
       <visual>
-        <origin xyz="3.35 0.0 0.0"/>
+        <origin xyz="0 0.0 0.0"/>
         <geometry>
           <mesh filename="package://abb_irbt6004_670_support/meshes/abb_irbt6004_670/visual/axis.stl"/>
@@ -15,5 +15,5 @@
       </visual>
       <collision>
-        <origin xyz="3.35 0.0 0.0"/>
+        <origin xyz="0 0.0 0.0"/>
         <geometry>
           <mesh filename="package://abb_irbt6004_670_support/meshes/abb_irbt6004_670/collision/axis.stl"/>
@@ -26,5 +26,5 @@
       <origin xyz="0 0 0.05" rpy="0 0 0 "/> <!--track origin or translation from origin-->
       <axis   xyz="1 0 0"/>
-      <limit lower="0" upper="6.700" effort="100000" velocity="2.618" />  <!--track limits or length-->
+      <limit lower="-3.35" upper="3.35" effort="100000" velocity="2.618" />  <!--track limits or length-->
       <dynamics damping="0.2" friction="0" />
     </joint>
