Commit message: MISC minor changes for the urdfs axes rotations

File: robot_files/abb_irb_6700_track_irtb_6004/4_urdfs/abb_irbt6004_670_support/urdf/abb_irb6700_175_305_ibois.xacro (robot description, xacro)
@@ -6,5 +6,5 @@
       <parent link="world" />
       <child link = "rob1_axis" />
-      <origin xyz="0.0 0.0 0.0" rpy="0.0 0.0 0.0" />
+      <origin xyz="-3.35 0.0 0.0" rpy="0.0 0.0 0.0" />
   </joint>
   <xacro:abb_irb6700_175_305_ibois prefix="rob1_" />

File: robot_files/abb_irb_6700_track_irtb_6004/4_urdfs/abb_irbt6004_670_support/urdf/abb_irb6700_175_305_ibois_macro.xacro (robot description, xacro)
@@ -10,5 +10,5 @@
       <parent link="${prefix}pedestal"/>
       <child  link="${prefix}base_link"/>
-      <origin xyz="0 0 0 " rpy="0 0 0 "/> <!--rotation of robot pedestal-->
+      <origin xyz="0 0 0 " rpy="0 0 -1.57079632679489661923 "/> <!--rotation of robot pedestal 3.14159265358979323846 1.57079632679489661923-->
       <dynamics damping="0.2" friction="0" />
     </joint>

File: robot_files/abb_irb_6700_track_irtb_6004_2x/4_urdfs/abb_irbt6004_670_support/urdf/abb_irb6700_175_305_crcl_macro.xacro (robot description, xacro)
@@ -10,5 +10,5 @@
       <parent link="${prefix}pedestal"/>
       <child  link="${prefix}base_link"/>
-      <origin xyz="0 0 0 " rpy="0 0 3.14159265358979323846 "/> <!--rotation of robot pedestal-->
+      <origin xyz="0 0 0 " rpy="0 0 1.57079632679 "/> <!--rotation of robot pedestal 1.57079632679 3.14159265358979323846-->
       <dynamics damping="0.2" friction="0" />
     </joint>

File: robot_files/abb_irb_6700_track_irtb_6004_2x/4_urdfs/abb_irbt6004_670_support/urdf/abb_irb6700_175_305_ibois_macro.xacro (robot description, xacro)
@@ -10,5 +10,5 @@
       <parent link="${prefix}pedestal"/>
       <child  link="${prefix}base_link"/>
-      <origin xyz="0 0 0 " rpy="0 0 0 "/> <!--rotation of robot pedestal-->
+      <origin xyz="0 0 0 " rpy="0 0 1.57079632679 "/> <!--rotation of robot pedestal-->
       <dynamics damping="0.2" friction="0" />
     </joint>

File: robot_files/abb_irb_6700_track_irtb_6004_2x/4_urdfs/abb_irbt6004_670_support/urdf/abb_irb6700_175_305_ibois_tworobots.xacro (robot description, xacro)
@@ -8,5 +8,5 @@
       <parent link="world" />
       <child link = "rob1_axis" />
-      <origin xyz="0 -1.5 0.0" rpy="0.0 0.0 0.0" /> <!--translation of the track-->
+      <origin xyz="-3.35 -1.5 0.0" rpy="0.0 0.0 0.0" /> <!--translation of the track-->
   </joint>
   <xacro:abb_irb6700_175_305_ibois prefix="rob1_" /> <!--robot with different base rotation-->
@@ -14,5 +14,5 @@
       <parent link="world" />
       <child link = "rob2_axis" />
-      <origin xyz="0 1.5 0.0" rpy="0.0 0.0 0" /> <!--translation of the track-->
+      <origin xyz="3.35 1.5 0.0" rpy="0.0 0.0 3.14159265358979323846" /> <!--translation of the track-->
   </joint>
   <xacro:abb_irb6700_175_305_crcl prefix="rob2_" /> <!--robot with different base rotation-->

File: robot_files/abb_irb_6700_track_irtb_6004_2x/4_urdfs/abb_irbt6004_670_support/urdf/abb_irbt6004_670.xacro (robot description, xacro)
@@ -8,5 +8,5 @@
       </inertial>
       <visual>
-        <origin xyz="0 0.0 0.0"/>
+        <origin xyz="3.35 0.0 0.0"/> <!--if x is zero the robot origin is at the center-->
         <geometry>
           <mesh filename="package://abb_irbt6004_670_support/meshes/abb_irbt6004_670/visual/axis.stl"/>
@@ -15,5 +15,5 @@
       </visual>
       <collision>
-        <origin xyz="0 0.0 0.0"/>
+        <origin xyz="3.35 0.0 0.0"/> <!--if x is zero the robot origin is at the center-->
         <geometry>
           <mesh filename="package://abb_irbt6004_670_support/meshes/abb_irbt6004_670/collision/axis.stl"/>
@@ -26,5 +26,5 @@
       <origin xyz="0 0 0.05" rpy="0 0 0 "/> <!--track origin or translation from origin-->
       <axis   xyz="1 0 0"/>
-      <limit lower="-3.35" upper="3.35" effort="100000" velocity="2.618" />  <!--track limits or length-->
+      <limit lower="0" upper="6.7" effort="100000" velocity="2.618" />  <!--track limits or length-->
       <dynamics damping="0.2" friction="0" />
     </joint>

Commit message: FIX update urdf

File: robot_files/abb_irb_6700_track_irtb_6004/4_urdfs/abb_irbt6004_670_support/urdf/abb_irb6700_175_305_ibois.xacro (robot description, xacro)
@@ -6,5 +6,5 @@
       <parent link="world" />
       <child link = "rob1_axis" />
-      <origin xyz="-3.35 0.0 0.0" rpy="0.0 0.0 0.0" />
+      <origin xyz="0 0.0 0.0" rpy="0.0 0.0 3.14159265358979323846" />
   </joint>
   <xacro:abb_irb6700_175_305_ibois prefix="rob1_" />

File: robot_files/abb_irb_6700_track_irtb_6004/4_urdfs/abb_irbt6004_670_support/urdf/abb_irb6700_175_305_ibois_macro.xacro (robot description, xacro)
@@ -10,5 +10,5 @@
       <parent link="${prefix}pedestal"/>
       <child  link="${prefix}base_link"/>
-      <origin xyz="0 0 0 " rpy="0 0 -1.57079632679489661923 "/> <!--rotation of robot pedestal 3.14159265358979323846 1.57079632679489661923-->
+      <origin xyz="0 0 0 " rpy="0 0 1.57079632679489661923 "/> <!--rotation of robot pedestal 3.14159265358979323846 1.57079632679489661923-->
       <dynamics damping="0.2" friction="0" />
     </joint>

File: robot_files/abb_irb_6700_track_irtb_6004/4_urdfs/abb_irbt6004_670_support/urdf/abb_irbt6004_670.xacro (robot description, xacro)
@@ -8,5 +8,5 @@
       </inertial>
       <visual>
-        <origin xyz="3.35 0.0 0.0"/>
+        <origin xyz="-3.35 0.0 0.0" />
         <geometry>
           <mesh filename="package://abb_irbt6004_670_support/meshes/abb_irbt6004_670/visual/axis.stl"/>
@@ -15,5 +15,5 @@
       </visual>
       <collision>
-        <origin xyz="3.35 0.0 0.0"/>
+        <origin xyz="-3.35 0.0 0.0"/>
         <geometry>
           <mesh filename="package://abb_irbt6004_670_support/meshes/abb_irbt6004_670/collision/axis.stl"/>
@@ -24,5 +24,5 @@
       <parent link="${prefix}axis"/>
       <child  link="${prefix}pedestal"/>
-      <origin xyz="0 0 0.05" rpy="0 0 0 "/> <!--track origin or translation from origin-->
+      <origin xyz="0 0 0.05" rpy="0 0 3.14159265358979323846 "/> <!--track origin or translation from origin-->
       <axis   xyz="1 0 0"/>
       <limit lower="0" upper="6.700" effort="100000" velocity="2.618" />  <!--track limits or length-->
