Commit message: ADD update grasshopper file

File: robot_files/abb_irb_6700_track_irtb_6004/2_docker/abb_irbt6004_670_support/urdf/abb_irbt6004_670.xacro (robot description, xacro)
@@ -8,5 +8,5 @@
       </inertial>
       <visual>
-        <origin xyz="3.35 0.0 0.0"/>
+        <origin xyz="-3.35 0.0 0.0" />
         <geometry>
           <mesh filename="package://abb_irbt6004_670_support/meshes/abb_irbt6004_670/visual/axis.stl"/>
@@ -15,5 +15,5 @@
       </visual>
       <collision>
-        <origin xyz="3.35 0.0 0.0"/>
+        <origin xyz="-3.35 0.0 0.0"/>
         <geometry>
           <mesh filename="package://abb_irbt6004_670_support/meshes/abb_irbt6004_670/collision/axis.stl"/>
@@ -24,5 +24,6 @@
       <parent link="${prefix}axis"/>
       <child  link="${prefix}pedestal"/>
-      <origin xyz="0 0 0.05" rpy="0 0 0 "/> <!--track origin or translation from origin-->
+      <!-- <origin xyz="0 0 0.05" rpy="0 0 3.14159265358979323846 "/> track origin or translation from origin -0.287 -1.919 -46.435 -->
+      <origin xyz="0.0000 0 0.05" rpy="0 0 3.14159265358979323846 "/> <!--track origin or translation from origin -0.287 -1.919 -46.435 -->
       <axis   xyz="1 0 0"/>
       <limit lower="0" upper="6.700" effort="100000" velocity="2.618" />  <!--track limits or length-->

Commit message: Update URDF and FK

File: robot_files/abb_irb_6700_track_irtb_6004/2_docker/abb_irbt6004_670_support/urdf/abb_irbt6004_670.xacro (robot description, xacro)
@@ -25,5 +25,5 @@
       <child  link="${prefix}pedestal"/>
       <!-- <origin xyz="0 0 0.05" rpy="0 0 3.14159265358979323846 "/> track origin or translation from origin -0.287 -1.919 -46.435 -->
-      <origin xyz="0.0000 0 0.05" rpy="0 0 3.14159265358979323846 "/> <!--track origin or translation from origin -0.287 -1.919 -46.435 -->
+      <origin xyz="-0.0000518 0.0006 0.0042" rpy="0 0.000312 3.14159265358979323846+0.000443"/> <!--track origin or translation from origin -0.287 -1.919 -46.435 -->
       <axis   xyz="1 0 0"/>
       <limit lower="0" upper="6.700" effort="100000" velocity="2.618" />  <!--track limits or length-->

Commit message: io python code

File: robot_files/abb_irb_6700_track_irtb_6004/2_docker/abb_irbt6004_670_support/urdf/abb_irbt6004_670.xacro (robot description, xacro)
@@ -25,5 +25,5 @@
       <child  link="${prefix}pedestal"/>
       <!-- <origin xyz="0 0 0.05" rpy="0 0 3.14159265358979323846 "/> track origin or translation from origin -0.287 -1.919 -46.435 -->
-      <origin xyz="-0.0000518 0.0006 0.0042" rpy="0 0.000312 3.14159265358979323846+0.000443"/> <!--track origin or translation from origin -0.287 -1.919 -46.435 -->
+      <origin xyz="-0.0000518 0.0006 0.0042" rpy="0 0.000312 3.14159265358979323846"/> <!--track origin or translation from origin -0.287 -1.919 -46.435  0 0.000312 3.14159265358979323846+0.000443     -->
       <axis   xyz="1 0 0"/>
       <limit lower="0" upper="6.700" effort="100000" velocity="2.618" />  <!--track limits or length-->

File: robot_files/abb_irb_6700_track_irtb_6004/4_urdfs/abb_irbt6004_670_support/urdf/abb_irbt6004_670.xacro (robot description, xacro)
@@ -24,5 +24,5 @@
       <parent link="${prefix}axis"/>
       <child  link="${prefix}pedestal"/>
-      <origin xyz="0 0 0.05" rpy="0 0 3.14159265358979323846 "/> <!--track origin or translation from origin-->
+      <origin xyz="0 0 0.05" rpy="0 0 3.14159 "/> <!--track origin or translation from origin 3.14159265358979323846 -->
       <axis   xyz="1 0 0"/>
       <limit lower="0" upper="6.700" effort="100000" velocity="2.618" />  <!--track limits or length-->

Commit message: Update URDF with Track Calibration Data
0504 calibration result, JW's version of motion planning,

File: robot_files/abb_irb_6700_track_irtb_6004/2_docker/abb_irbt6004_670_support/urdf/abb_irbt6004_670.xacro (robot description, xacro)
@@ -8,5 +8,5 @@
       </inertial>
       <visual>
-        <origin xyz="-3.35 0.0 0.0" />
+        <origin xyz="3.35 0.0 0.0" />
         <geometry>
           <mesh filename="package://abb_irbt6004_670_support/meshes/abb_irbt6004_670/visual/axis.stl"/>
@@ -15,5 +15,5 @@
       </visual>
       <collision>
-        <origin xyz="-3.35 0.0 0.0"/>
+        <origin xyz="3.35 0.0 0.0"/>
         <geometry>
           <mesh filename="package://abb_irbt6004_670_support/meshes/abb_irbt6004_670/collision/axis.stl"/>
@@ -24,6 +24,5 @@
       <parent link="${prefix}axis"/>
       <child  link="${prefix}pedestal"/>
-      <!-- <origin xyz="0 0 0.05" rpy="0 0 3.14159265358979323846 "/> track origin or translation from origin -0.287 -1.919 -46.435 -->
-      <origin xyz="-0.0000518 0.0006 0.0042" rpy="0 0.000312 3.14159265358979323846"/> <!--track origin or translation from origin -0.287 -1.919 -46.435  0 0.000312 3.14159265358979323846+0.000443     -->
+      <origin xyz="0 0 0" rpy="0 0 0"/> <!--track origin or translation from origin-->
       <axis   xyz="1 0 0"/>
       <limit lower="0" upper="6.700" effort="100000" velocity="2.618" />  <!--track limits or length-->

File: robot_files/abb_irb_6700_track_irtb_6004/4_urdfs/abb_irbt6004_670_support/urdf/abb_irbt6004_670.xacro (robot description, xacro)
@@ -8,5 +8,5 @@
       </inertial>
       <visual>
-        <origin xyz="-3.35 0.0 0.0" />
+        <origin xyz="3.35 0.0 0.0" />
         <geometry>
           <mesh filename="package://abb_irbt6004_670_support/meshes/abb_irbt6004_670/visual/axis.stl"/>
@@ -15,5 +15,5 @@
       </visual>
       <collision>
-        <origin xyz="-3.35 0.0 0.0"/>
+        <origin xyz="3.35 0.0 0.0"/>
         <geometry>
           <mesh filename="package://abb_irbt6004_670_support/meshes/abb_irbt6004_670/collision/axis.stl"/>
@@ -24,5 +24,5 @@
       <parent link="${prefix}axis"/>
       <child  link="${prefix}pedestal"/>
-      <origin xyz="0 0 0.05" rpy="0 0 3.14159 "/> <!--track origin or translation from origin 3.14159265358979323846 -->
+      <origin xyz="0 0 0" rpy="0 0 0"/> <!--track origin or translation from origin-->
       <axis   xyz="1 0 0"/>
       <limit lower="0" upper="6.700" effort="100000" velocity="2.618" />  <!--track limits or length-->
