Commit message: Update the docker for aurora

File: robot_files/abb_irb_6700_track_irtb_6004/2_docker/abb_irbt6004_670_moveit_config/config/gazebo_aurora.urdf (robot description, URDF)
Before this commit: robot abb_irb6700_175_305_ibois, 15 links, 14 joints
Links:
- link rob1_axis: geometry collision mesh filename=package://abb_irbt6004_670_moveit_config/meshes/abb_irbt600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; visual mesh filename=package://abb_irbt6004_670_moveit_config/meshes/abb_irbt600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
- link rob1_pedestal: geometry collision mesh filename=package://abb_irbt6004_670_moveit_config/meshes/abb_irbt600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; visual mesh filename=package://abb_irbt6004_670_moveit_config/meshes/abb_irbt600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

File: robot_files/abb_irb_6700_track_irtb_6004/2_docker/abb_irbt6004_670_moveit_config/urdf/abb_irb6700_175_305_ibois.xacro (robot description, xacro)
@@ -1,5 +1,5 @@
 <?xml version="1.0"?>
-<robot name="abb_irb6700_175_305_ibois" xmlns:xacro="http://ros.org/wiki/xacro">
-  <xacro:include filename="$(find abb_irbt6004_670_support)/urdf/abb_irb6700_175_305_ibois_macro.xacro"/>
+<robot name="aurora" xmlns:xacro="http://ros.org/wiki/xacro">
+  <xacro:include filename="$(find abb_irbt6004_670_moveit_config)/urdf/abb_irb6700_175_305_ibois_macro.xacro"/>
   <link name="world" />
   <joint name="world_joint" type="fixed">

File: robot_files/abb_irb_6700_track_irtb_6004/2_docker/abb_irbt6004_670_moveit_config/urdf/abb_irb6700_175_305_ibois_macro.xacro (robot description, xacro)
@@ -2,8 +2,7 @@
 <robot xmlns:xacro="http://wiki.ros.org/xacro">
   <xacro:macro name="abb_irb6700_175_305_ibois" params="prefix" >
-  <!--<xacro:macro name="abb_irb6700_175_305_ibois" params="prefix prefix_notused" >-->
     <xacro:include filename="$(find abb_resources)/urdf/common_materials.xacro"/>
     <xacro:include filename="$(find abb_irb6700_support)/urdf/irb6700_175_305_macro.xacro"/>
-    <xacro:include filename="$(find abb_irbt6004_670_support)/urdf/abb_irbt6004_670.xacro"/>
+    <xacro:include filename="$(find abb_irbt6004_670_moveit_config)/urdf/abb_irbt6004_670.xacro"/>
     <xacro:abb_irbt6004_670 prefix="${prefix}" />
     <joint name="${prefix}abb_joint" type="fixed">

File: robot_files/abb_irb_6700_track_irtb_6004/2_docker/abb_irbt6004_670_moveit_config/urdf/abb_irbt6004_670.xacro (robot description, xacro)
@@ -10,5 +10,5 @@
         <origin xyz="3.35 0.0 0.0" />
         <geometry>
-          <mesh filename="package://abb_irbt6004_670_support/meshes/abb_irbt6004_670/visual/axis.stl"/>
+          <mesh filename="package://abb_irbt6004_670_moveit_config/meshes/abb_irbt6004_670/visual/axis.stl"/>
         </geometry>
         <xacro:material_abb_white />
@@ -17,5 +17,5 @@
         <origin xyz="3.35 0.0 0.0"/>
         <geometry>
-          <mesh filename="package://abb_irbt6004_670_support/meshes/abb_irbt6004_670/collision/axis.stl"/>
+          <mesh filename="package://abb_irbt6004_670_moveit_config/meshes/abb_irbt6004_670/collision/axis.stl"/>
         </geometry>
       </collision>
@@ -37,5 +37,5 @@
       <visual>
         <geometry>
-          <mesh filename="package://abb_irbt6004_670_support/meshes/abb_irbt6004_670/visual/pedestal_250.stl"/>
+          <mesh filename="package://abb_irbt6004_670_moveit_config/meshes/abb_irbt6004_670/visual/pedestal_250.stl"/>
         </geometry>
         <xacro:material_abb_white />
@@ -43,5 +43,5 @@
       <collision>
         <geometry>
-          <mesh filename="package://abb_irbt6004_670_support/meshes/abb_irbt6004_670/collision/pedestal_250.stl"/>
+          <mesh filename="package://abb_irbt6004_670_moveit_config/meshes/abb_irbt6004_670/collision/pedestal_250.stl"/>
         </geometry>
       </collision>
